File: Atmega328p.sch (KiCad schematic (older format))
At the start: 4 parts

Commit message: Components
Crystal Circuit is done
USB is partially finished
Parts:
- removed U?: ATmega32U4-AU, Package_QFP:TQFP-44_10x10mm_P0.8mm, symbol MCU_Microchip_ATmega:ATmega32U4-AU
- removed Y?: Crystal, symbol Device:Crystal
- added C3: 1uF, symbol Device:CP1
- added J1: USB_B_Mini, symbol Connector:USB_B_Mini
- added U1: ATmega32U4-MU, Package_DFN_QFN:QFN-44-1EP_7x7mm_P0.5mm_EP5.4x5.4mm, symbol MCU_Microchip_ATmega:ATmega32U4-MU
- added U2: MCP1825, symbol Regulator_LinearV2:MCP1825
- added Y?: 12.88455, symbol Device:Crystal_GND24
- C1, C2: renamed from C?; value CAP -> 25pF
Connections:
- net labels added: GND, VCC
- wire segments 10 -> 23
Changed lines of the file:
@@
 EESchema Schematic File Version 4
+LIBS:Atmega328p-cache
 EELAYER 26 0
 EELAYER END
@@
 Comment4 ""
 $EndDescr
-$Comp
-L MCU_Microchip_ATmega:ATmega32U4-AU U?
-U 1 1 5B76E964
-P 4300 3900
-F 0 "U?" H 4300 2014 50  0000 C CNN
-F 1 "ATmega32U4-AU" H 4300 1923 50  0000 C CNN
-F 2 "Package_QFP:TQFP-44_10x10mm_P0.8mm" H 4300 3900 50  0001 C CIN
-F 3 "http://ww1.microchip.com/downloads/en/DeviceDoc/Atmel-7766-8-bit-AVR-ATmega16U4-32U4_Datasheet.pdf" H 4300 3900 50  0001 C CNN
-	1    4300 3900
-	1    0    0    -1
-$EndComp
-$Comp
-L Device:Crystal Y?
-U 1 1 5B76E9D3
-P 3350 2700
-F 0 "Y?" V 3304 2569 50  0000 R CNN
-F 1 "Crystal" V 3395 2569 50  0000 R CNN
-F 2 "" H 3350 2700 50  0001 C CNN
-F 3 "~" H 3350 2700 50  0001 C CNN
-	1    3350 2700
-	0    1    1    0
-$EndComp
-Wire Wire Line
-	3700 2600 3500 2600
-Wire Wire Line
-	3500 2600 3500 2550
-Wire Wire Line
-	3500 2550 3350 2550
-Wire Wire Line
-	3700 2800 3500 2800
-Wire Wire Line
-	3500 2800 3500 2850
-Wire Wire Line
-	3500 2850 3350 2850
-$Comp
-L pspice:CAP C?
+Wire Wire Line
+	5450 2300 5250 2300
+Wire Wire Line
+	5250 2300 5250 2250
+Wire Wire Line
+	5450 2500 5250 2500
+Wire Wire Line
+	5250 2500 5250 2550
+$Comp
+L pspice:CAP C1
 U 1 1 5B76EBAD
-P 2850 2500
-F 0 "C?" V 2535 2500 50  0000 C CNN
-F 1 "CAP" V 2626 2500 50  0000 C CNN
-F 2 "" H 2850 2500 50  0001 C CNN
-F 3 "" H 2850 2500 50  0001 C CNN
-	1    2850 2500
-	0    1    1    0
-$EndComp
-$Comp
-L pspice:CAP C?
+P 4550 2200
+F 0 "C1" V 4235 2200 50  0000 C CNN
+F 1 "25pF" V 4326 2200 50  0000 C CNN
+F 2 "" H 4550 2200 50  0001 C CNN
+F 3 "" H 4550 2200 50  0001 C CNN
+	1    4550 2200
+	0    1    1    0
+$EndComp
+Wire Wire Line
+	4900 2250 4900 2200
+Wire Wire Line
+	4900 2550 4900 2600
+$Comp
+L power:GND #PWR?
+U 1 1 5B76F376
+P 4300 2400
+F 0 "#PWR?" H 4300 2150 50  0001 C CNN
+F 1 "GND" V 4305 2272 50  0000 R CNN
+F 2 "" H 4300 2400 50  0001 C CNN
+F 3 "" H 4300 2400 50  0001 C CNN
+	1    4300 2400
+	0    1    1    0
+$EndComp
+Wire Wire Line
+	4300 2200 4300 2400
+Wire Wire Line
+	4300 2600 4300 2400
+Connection ~ 4300 2400
+$Comp
+L pspice:CAP C2
 U 1 1 5B76EC09
-P 2850 2900
-F 0 "C?" V 3073 2900 50  0000 C CNN
-F 1 "CAP" V 3164 2900 50  0000 C CNN
-F 2 "" H 2850 2900 50  0001 C CNN
-F 3 "" H 2850 2900 50  0001 C CNN
-	1    2850 2900
-	0    1    1    0
-$EndComp
-Wire Wire Line
-	3350 2550 3350 2500
-Wire Wire Line
-	3350 2500 3100 2500
-Connection ~ 3350 2550
-Wire Wire Line
-	3350 2850 3350 2900
-Wire Wire Line
-	3350 2900 3100 2900
-Connection ~ 3350 2850
+P 4550 2600
+F 0 "C2" V 4773 2600 50  0000 C CNN
+F 1 "25pF" V 4864 2600 50  0000 C CNN
+F 2 "" H 4550 2600 50  0001 C CNN
+F 3 "" H 4550 2600 50  0001 C CNN
+	1    4550 2600
+	0    1    1    0
+$EndComp
+Wire Wire Line
+	4900 2250 5250 2250
+Wire Wire Line
+	4900 2550 5250 2550
+$Comp
+L MCU_Microchip_ATmega:ATmega32U4-MU U1
+U 1 1 5B77029B
+P 6050 3600
+F 0 "U1" H 6400 1850 50  0000 C CNN
+F 1 "ATmega32U4-MU" H 6400 1750 50  0000 C CNN
+F 2 "Package_DFN_QFN:QFN-44-1EP_7x7mm_P0.5mm_EP5.4x5.4mm" H 6050 3600 50  0001 C CIN
+F 3 "http://ww1.microchip.com/downloads/en/DeviceDoc/Atmel-7766-8-bit-AVR-ATmega16U4-32U4_Datasheet.pdf" H 6050 3600 50  0001 C CNN
+	1    6050 3600
+	1    0    0    -1
+$EndComp
+$Comp
+L power:GND #PWR?
+U 1 1 5B770886
+P 5700 5450
+F 0 "#PWR?" H 5700 5200 50  0001 C CNN
+F 1 "GND" V 5705 5322 50  0000 R CNN
+F 2 "" H 5700 5450 50  0001 C CNN
+F 3 "" H 5700 5450 50  0001 C CNN
+	1    5700 5450
+	0    1    1    0
+$EndComp
+Wire Wire Line
+	5950 5400 5950 5450
+Wire Wire Line
+	6050 5400 6050 5450
+Wire Wire Line
+	5700 5450 5950 5450
+Connection ~ 5950 5450
+Wire Wire Line
+	5950 5450 6050 5450
+$Comp
+L Device:Crystal_GND24 Y?
+U 1 1 5B77432D
+P 4900 2400
+F 0 "Y?" V 5150 2400 50  0000 L CNN
+F 1 "12.88455" V 5250 2200 50  0000 L CNN
+F 2 "" H 4900 2400 50  0001 C CNN
+F 3 "~" H 4900 2400 50  0001 C CNN
+	1    4900 2400
+	0    1    1    0
+$EndComp
+Connection ~ 4900 2250
+Connection ~ 4900 2550
+Wire Wire Line
+	4900 2200 4800 2200
+Wire Wire Line
+	4900 2600 4800 2600
+$Comp
+L power:GND #PWR?
+U 1 1 5B77507D
+P 3150 3650
+F 0 "#PWR?" H 3150 3400 50  0001 C CNN
+F 1 "GND" H 3155 3477 50  0000 C CNN
+F 2 "" H 3150 3650 50  0001 C CNN
+F 3 "" H 3150 3650 50  0001 C CNN
+	1    3150 3650
+	1    0    0    -1
+$EndComp
+$Comp
+L Device:CP1 C3
+U 1 1 5B777265
+P 3000 2950
+F 0 "C3" V 3252 2950 50  0000 C CNN
+F 1 "1uF" V 3161 2950 50  0000 C CNN
+F 2 "" H 3000 2950 50  0001 C CNN
+F 3 "~" H 3000 2950 50  0001 C CNN
+	1    3000 2950
+	0    -1   -1   0
+$EndComp
+$Comp
+L power:GND #PWR?
+U 1 1 5B7772D1
+P 3150 2950
+F 0 "#PWR?" H 3150 2700 50  0001 C CNN
+F 1 "GND" H 3155 2777 50  0000 C CNN
+F 2 "" H 3150 2950 50  0001 C CNN
+F 3 "" H 3150 2950 50  0001 C CNN
+	1    3150 2950
+	0    -1   -1   0
+$EndComp
+$Comp
+L Connector:USB_B_Mini J1
+U 1 1 5B774950
+P 2500 4050
+F 0 "J1" H 2555 4517 50  0000 C CNN
+F 1 "USB_B_Mini" H 1950 4000 50  0000 C CNN
+F 2 "" H 2650 4000 50  0001 C CNN
+F 3 "~" H 2650 4000 50  0001 C CNN
+	1    2500 4050
+	1    0    0    -1
+$EndComp
+Wire Wire Line
+	2800 3850 2850 3850
+Wire Wire Line
+	2850 3850 2850 3350
+$Comp
+L Regulator_LinearV2:MCP1825 U2
+U 1 1 5B77AA97
+P 3150 3400
+F 0 "U2" H 3150 3692 50  0000 C CNN
+F 1 "MCP1825" H 3150 3601 50  0000 C CNN
+F 2 "" H 2950 3600 50  0001 C CNN
+F 3 "" H 2950 3600 50  0001 C CNN
+	1    3150 3400
+	1    0    0    -1
+$EndComp
+Wire Wire Line
+	2850 3350 2850 2950
+Wire Wire Line
+	5950 1650 5950 1800
+Connection ~ 2850 3350
+Connection ~ 2850 2950
+Wire Wire Line
+	2850 2950 2850 2650
+Wire Wire Line
+	5300 2950 5300 2900
+Wire Wire Line
+	5300 2900 5450 2900
+$Comp
+L power:VCC #PWR?
+U 1 1 5B783C24
+P 6050 1800
+F 0 "#PWR?" H 6050 1650 50  0001 C CNN
+F 1 "VCC" H 6067 1973 50  0000 C CNN
+F 2 "" H 6050 1800 50  0001 C CNN
+F 3 "" H 6050 1800 50  0001 C CNN
+	1    6050 1800
+	1    0    0    -1
+$EndComp
+$Comp
+L power:GND #PWR?
+U 1 1 5B783C7E
+P 4900 4100
+F 0 "#PWR?" H 4900 3850 50  0001 C CNN
+F 1 "GND" H 4905 3927 50  0000 C CNN
+F 2 "" H 4900 4100 50  0001 C CNN
+F 3 "" H 4900 4100 50  0001 C CNN
+	1    4900 4100
+	1    0    0    -1
+$EndComp
 $EndSCHEMATC

Commit message: Board V1.0
Parts:
- removed J1: USB_B_Mini, symbol Connector:USB_B_Mini
- removed U1: ATmega32U4-MU, Package_DFN_QFN:QFN-44-1EP_7x7mm_P0.5mm_EP5.4x5.4mm, symbol MCU_Microchip_ATmega:ATmega32U4-MU
- removed U2: MCP1825, symbol Regulator_LinearV2:MCP1825
- added C4, C5, C6, C7: 0.1uF, symbol Device:CP1_Small
- added IC1: ATMEGA32U4, symbol freetronics_schematic:ATMEGA32U4
- added J1: AREF, symbol Connector:Conn_01x01_Female
- added J2: RST, symbol Connector:Conn_01x01_Female
- added J3: VCC, symbol Connector:Conn_01x01_Female
- added J4: GND, symbol Connector:Conn_01x01_Female
- added J5, J? (x2): Conn_01x12_Female, symbol Connector:Conn_01x12_Female
- added J6: Conn_01x08_Female, symbol Connector:Conn_01x08_Female
- added P1: USB_4PIN_NO_SHELL, symbol freetronics_schematic:USB_4PIN_NO_SHELL
- added R1, R2: 22ohm, symbol Device:R
- added R3: 1k, symbol Device:R
- added SW1: SW_Push, symbol Switch:SW_Push
- gave numbers to parts that had none: 1
Connections:
- net labels added: AREF, B0, B1, B2, B3, B4, B5, B6, B7, C6, C7, D0, D1, D2, D3, D4, D5, E6, F0, F1, F4, F5, F6, F7
- wire segments 23 -> 82

Commit message: Footprint Assosciation
Parts:
- removed J6: Conn_01x08_Female, symbol Connector:Conn_01x08_Female
- removed J?: Conn_01x12_Female, symbol Connector:Conn_01x12_Female
- C1, C2, C3, C4, C5, C6, C7: footprint (none) -> Capacitor_SMD:C_0805_2012Metric
- IC1: footprint (none) -> Package_QFP:TQFP-44_10x10mm_P0.8mm
- J1, J2, J3, J4: footprint (none) -> Connector_PinHeader_1.00mm:PinHeader_1x01_P1.00mm_Vertical
- J5: footprint (none) -> Connector_PinHeader_1.00mm:PinHeader_1x12_P1.00mm_Vertical
- J7: renamed from J?; footprint (none) -> Connector_PinHeader_1.00mm:PinHeader_1x12_P1.00mm_Vertical
- P1: footprint (none) -> Connector_USB:USB_Mini-B_Lumberg_2486_01_Horizontal
- R1, R2, R3: footprint (none) -> Resistor_SMD:R_0805_2012Metric
- SW1: footprint (none) -> Button_Switch_THT:SW_PUSH_6mm_H4.3mm
- Y1: footprint (none) -> Crystal:Crystal_SMD_3225-4Pin_3.2x2.5mm
